Commit message: Solved problem on rviz

File: description/robot_core.xacro (robot description, xacro)
@@ -86,5 +86,5 @@
         </xacro:inertial_cylinder>
     </link>
-    <joint name="left_wheel_joint" type="fixed">
+    <joint name="left_wheel_joint" type="continuous">
         <parent link="base_link"/>
         <child link="left_wheel"/>
@@ -112,8 +112,8 @@
         </xacro:inertial_cylinder>
     </link>
-    <joint name="right_wheel_joint" type="fixed">
+    <joint name="right_wheel_joint" type="continuous">
         <parent link="base_link"/>
         <child link="right_wheel"/>
-        <origin xyz="0 ${-wheel_offset_y-10} 0" rpy="${pi/2} 0 0" />
+        <origin xyz="0 ${-wheel_offset_y} 0" rpy="${pi/2} 0 0" />
         <axis xyz="0 0 -1"/>
     </joint>

File: description/ros2_control.xacro (robot description, xacro)
@@ -56,6 +56,6 @@
     <gazebo>
         <plugin name="gazebo_ros2_control" filename="libgazebo_ros2_control.so">
-            <parameters>$(find articubot_one)/config/my_controllers.yaml</parameters>
-            <parameters>$(find articubot_one)/config/gaz_ros2_ctl_use_sim.yaml</parameters>
+            <parameters>$(find kilobot)/config/my_controllers.yaml</parameters>
+            <parameters>$(find kilobot)/config/gaz_ros2_ctl_use_sim.yaml</parameters>
         </plugin>
     </gazebo>
